Commit message: Some changes for the successful compilation

File: hsmakata/hsmakata_description/robots/hsmakata.urdf.xacro (robot description, xacro)
@@ -63,5 +63,5 @@
     <parent link="top_plate" />
     <child link="kata_plate_link" />
-    <origin rpy="0 0 0" xyz="0.022 0 0.191" />
+    <origin rpy="0 0 0" xyz="-0.020 0 0.191" />
   </joint>
   <!-- **************************** -->

File: hsmakata/hsmakata_description/urdf/hsmakata.urdf (robot description, URDF)
Before this commit: robot hsmakata, 35 links, 34 joints
Links:
- link back_sonar: geometry collision box size=0.5 0.25 0.05; visual mesh filename=package://p2os_urdf/meshes/p3dx_meshes/back_sonar.stl
- link base_link: mass None -> 40.0; geometry collision mesh filename=package://p2os_urdf/meshes/p3at_meshes/chassis.stl; visual mesh filename=package://p2os_urdf/meshes/p3dx_meshes/chassis.stl
- link center_hubcap: geometry collision box size=0.05 0.05 0.05; visual mesh filename=package://p2os_urdf/meshes/p3dx_meshes/center_hubcap.stl
- link left_hub: geometry collision cylinder length=0.01 radius=0.09; visual mesh filename=package://p2os_urdf/meshes/p3dx_meshes/left_hubcap.stl
- link right_hub: geometry collision cylinder length=0.01 radius=0.09; visual mesh filename=package://p2os_urdf/meshes/p3dx_meshes/right_hubcap.stl
- link top_plate: mass None -> 0.01
Joints:
- joint base_top_joint: origin xyz=-0.045 0 0.234 rpy=0 0 0 -> xyz=-0.045 0 0.24 rpy=0 0 0
- joint kata_plate_joint: origin xyz=0.022 0 0.191 rpy=0 0 0 -> xyz=-0.020 0 0.191 rpy=0 0 0
